File: power_3V3.kicad_sch (KiCad schematic)
At the start: 3 parts, among them U10 TLV76033

Commit message: Move to SIM800C-DS and two SIM
Connections:
- net 3V3_OUT: now also U10.1 (VO); no longer U10.2 (VO)
- net 5V_IN: now also U10.2 (VI); no longer U10.3 (VI)
- net GNDD: now also U10.3 (GND); no longer U10.1 (GND)
