File: MCU.kicad_sch (KiCad schematic)
At the start: 40 parts, among them J10 Conn_01x05_Pin, J11 Conn_02x02_2.54, SW1 SM5-180UP-1, U9 STM32L072CBT6, Y1 4 MHz, Y2 32768 kHz

Commit message: Release candidate
Parts:
- JP6, JP7: footprint TestPoint:TestPoint_2Pads_Pitch2.54mm_Drill0.8mm -> Connector_PinHeader_2.54mm:PinHeader_1x02_P2.54mm_Vertical
Connections:
- net UART1_RX: now also J11.4 (Pin_4); no longer J11.2 (Pin_2)
- net UART1_TX: now also J11.2 (Pin_2); no longer J11.4 (Pin_4)
Other:
- moved on the sheet: J11
Changed lines of the file:
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@@
 (kicad_sch
-	(version 20260101)
+	(version 20260306)
 	(generator "eeschema")
 	(generator_version "10.0")
@@
 	)
 	(junction
-		(at 45.72 25.4)
+		(at 156.21 116.84)
 		(diameter 0)
 		(color 0 0 0 0)
 	)
 	(junction
-		(at 130.81 43.18)
+		(at 45.72 25.4)
 		(diameter 0)
 		(color 0 0 0 0)
 	)
 	(junction
-		(at 156.21 119.38)
+		(at 130.81 43.18)
 		(diameter 0)
 		(color 0 0 0 0)
 	)
 	(junction
-		(at 181.61 116.84)
+		(at 133.35 140.97)
 		(diameter 0)
 		(color 0 0 0 0)
 	)
 	(junction
-		(at 133.35 140.97)
+		(at 54.61 25.4)
 		(diameter 0)
 		(color 0 0 0 0)
 	)
 	(junction
-		(at 54.61 25.4)
+		(at 82.55 93.98)
 		(diameter 0)
 		(color 0 0 0 0)
 	)
 	(junction
-		(at 82.55 93.98)
+		(at 187.96 119.38)
 		(diameter 0)
 		(color 0 0 0 0)
@@
 	(wire
 		(pts
-			(xy 165.1 116.84) (xy 166.37 116.84)
-		)
-		(stroke
-			(width 0)
-			(type default)
-		)
-	)
-	(wire
-		(pts
-			(xy 187.96 128.27) (xy 187.96 116.84)
+			(xy 181.61 116.84) (xy 180.34 116.84)
 		)
 		(stroke
@@
 	(wire
 		(pts
-			(xy 181.61 106.68) (xy 181.61 116.84)
+			(xy 187.96 106.68) (xy 187.96 119.38)
 		)
 		(stroke
@@
 	(wire
 		(pts
+			(xy 180.34 119.38) (xy 187.96 119.38)
+		)
+		(stroke
+			(width 0)
+			(type default)
+		)
+	)
+	(wire
+		(pts
 			(xy 148.59 81.28) (xy 212.09 81.28)
 		)
@@
 	(wire
 		(pts
-			(xy 74.93 93.98) (xy 82.55 93.98)
+			(xy 156.21 116.84) (xy 156.21 130.81)
 		)
 		(stroke
@@
 	(wire
 		(pts
-			(xy 187.96 116.84) (xy 181.61 116.84)
+			(xy 74.93 93.98) (xy 82.55 93.98)
 		)
 		(stroke
@@
 	(wire
 		(pts
-			(xy 165.1 115.57) (xy 165.1 116.84)
+			(xy 181.61 115.57) (xy 181.61 116.84)
 		)
 		(stroke
@@
 	(wire
 		(pts
-			(xy 173.99 106.68) (xy 181.61 106.68)
+			(xy 173.99 106.68) (xy 187.96 106.68)
 		)
 		(stroke
@@
 	(wire
 		(pts
+			(xy 187.96 119.38) (xy 187.96 128.27)
+		)
+		(stroke
+			(width 0)
+			(type default)
+		)
+	)
+	(wire
+		(pts
 			(xy 133.35 53.34) (xy 133.35 55.88)
 		)
@@
 	(wire
 		(pts
-			(xy 156.21 119.38) (xy 166.37 119.38)
-		)
-		(stroke
-			(width 0)
-			(type default)
-		)
-	)
-	(wire
-		(pts
 			(xy 50.8 104.14) (xy 113.03 104.14)
 		)
@@
 	(wire
 		(pts
-			(xy 181.61 116.84) (xy 179.07 116.84)
-		)
-		(stroke
-			(width 0)
-			(type default)
-		)
-	)
-	(wire
-		(pts
 			(xy 36.83 35.56) (xy 45.72 35.56)
 		)
@@
 	(wire
 		(pts
-			(xy 179.07 119.38) (xy 181.61 119.38)
+			(xy 167.64 119.38) (xy 165.1 119.38)
 		)
 		(stroke
@@
 	(wire
 		(pts
+			(xy 156.21 116.84) (xy 167.64 116.84)
+		)
+		(stroke
+			(width 0)
+			(type default)
+		)
+	)
+	(wire
+		(pts
 			(xy 121.92 158.75) (xy 121.92 161.29)
 		)
@@
 	(wire
 		(pts
-			(xy 156.21 106.68) (xy 156.21 119.38)
-		)
-		(stroke
-			(width 0)
-			(type default)
-		)
-	)
-	(wire
-		(pts
 			(xy 110.49 109.22) (xy 113.03 109.22)
 		)
@@
 	(wire
 		(pts
-			(xy 156.21 130.81) (xy 156.21 119.38)
+			(xy 156.21 106.68) (xy 156.21 116.84)
 		)
 		(stroke
@@
 	(wire
 		(pts
-			(xy 181.61 119.38) (xy 181.61 123.19)
+			(xy 165.1 119.38) (xy 165.1 123.19)
 		)
 		(stroke
@@
 	)
 	(label "UART1_TX"
-		(at 173.99 106.68 0)
+		(at 176.53 106.68 0)
 		(effects
 			(font
@@
 		)
 	)
-	(label "UART1_RX"
-		(at 156.21 119.38 0)
-		(effects
-			(font
-				(size 1.27 1.27)
-			)
-			(justify left bottom)
-		)
-	)
 	(label "USB_D-"
 		(at 209.55 93.98 180)
@@
 		)
 	)
+	(label "UART1_RX"
+		(at 157.48 116.84 0)
+		(effects
+			(font
+				(size 1.27 1.27)
+			)
+			(justify left bottom)
+		)
+	)
 	(label "RS485_EN"
 		(at 209.55 99.06 180)
@@
 	(symbol
 		(lib_id "power:GNDD")
-		(at 181.61 123.19 0)
+		(at 165.1 123.19 0)
+		(mirror y)
 		(unit 1)
 		(body_style 1)
@@
 		(fields_autoplaced yes)
 		(property "Reference" "#PWR074"
-			(at 181.61 129.54 0)
+			(at 165.1 129.54 0)
 			(hide yes)
 			(show_name no)
@@
 		)
 		(property "Value" "GNDD"
-			(at 181.61 127 0)
+			(at 165.1 127 0)
 			(show_name no)
 			(do_not_autoplace no)
@@
 		)
 		(property "Footprint" ""
-			(at 181.61 123.19 0)
+			(at 165.1 123.19 0)
 			(hide yes)
 			(show_name no)
@@
 		)
 		(property "Datasheet" ""
-			(at 181.61 123.19 0)
+			(at 165.1 123.19 0)
 			(hide yes)
 			(show_name no)
@@
 		)
 		(property "Description" "Power symbol creates a global label with name \"GNDD\" , digital ground"
-			(at 181.61 123.19 0)
+			(at 165.1 123.19 0)
 			(hide yes)
 			(show_name no)
@@
 			)
 		)
-		(property "Footprint" "TestPoint:TestPoint_2Pads_Pitch2.54mm_Drill0.8mm"
+		(property "Footprint" "Connector_PinHeader_2.54mm:PinHeader_1x02_P2.54mm_Vertical"
 			(at 43.18 115.57 0)
 			(hide yes)
@@
 	(symbol
 		(lib_id "Connector_Generic:Conn_02x02_Counter_Clockwise")
-		(at 171.45 116.84 0)
+		(at 175.26 116.84 0)
+		(mirror y)
 		(unit 1)
 		(body_style 1)
@@
 		(dnp no)
 		(property "Reference" "J11"
-			(at 172.72 114.046 0)
+			(at 173.99 114.046 0)
 			(show_name no)
 			(do_not_autoplace no)
@@
 		)
 		(property "Value" "Conn_02x02_2.54"
-			(at 172.974 121.92 0)
+			(at 173.736 121.92 0)
 			(show_name no)
 			(do_not_autoplace no)
@@
 		)
 		(property "Footprint" "Connector_PinSocket_2.54mm:PinSocket_2x02_P2.54mm_Vertical"
-			(at 171.45 116.84 0)
+			(at 175.26 116.84 0)
 			(hide yes)
 			(show_name no)
@@
 		)
 		(property "Datasheet" ""
-			(at 171.45 116.84 0)
+			(at 175.26 116.84 0)
 			(hide yes)
 			(show_name no)
@@
 		)
 		(property "Description" "Generic connector, double row, 02x02, counter clockwise pin numbering scheme (similar to DIP package numbering), script generated (kicad-library-utils/schlib/autogen/connector/)"
-			(at 171.45 116.84 0)
+			(at 175.26 116.84 0)
 			(hide yes)
 			(show_name no)
@@
 		)
 		(property "Manufacturer" "CONNFLY ELECTRONIC CO. LTD"
-			(at 171.45 116.84 0)
+			(at 175.26 116.84 0)
 			(hide yes)
 			(show_name no)
@@
 		)
 		(property "MPN" "DS1023-2*2SF11"
-			(at 171.45 116.84 0)
+			(at 175.26 116.84 0)
 			(hide yes)
 			(show_name no)
@@
 	(symbol
 		(lib_id "power:+3.3V")
-		(at 165.1 115.57 0)
+		(at 181.61 115.57 0)
+		(mirror y)
 		(unit 1)
 		(body_style 1)
@@
 		(dnp no)
 		(property "Reference" "#PWR073"
-			(at 165.1 119.38 0)
+			(at 181.61 119.38 0)
 			(hide yes)
 			(show_name no)
@@
 		)
 		(property "Value" "+3V3"
-			(at 162.052 111.506 0)
+			(at 184.658 111.506 0)
 			(show_name no)
 			(do_not_autoplace no)
@@
 		)
 		(property "Footprint" ""
-			(at 165.1 115.57 0)
+			(at 181.61 115.57 0)
 			(hide yes)
 			(show_name no)
@@
 		)
 		(property "Datasheet" ""
-			(at 165.1 115.57 0)
+			(at 181.61 115.57 0)
 			(hide yes)
 			(show_name no)
@@
 		)
 		(property "Description" "Power symbol creates a global label with name \"+3.3V\""
-			(at 165.1 115.57 0)
+			(at 181.61 115.57 0)
 			(hide yes)
 			(show_name no)
@@
 			)
 		)
-		(property "Footprint" "TestPoint:TestPoint_2Pads_Pitch2.54mm_Drill0.8mm"
+		(property "Footprint" "Connector_PinHeader_2.54mm:PinHeader_1x02_P2.54mm_Vertical"
 			(at 91.44 49.53 0)
 			(hide yes)

Commit message: Proproduction version
Parts:
- removed C25, C26, C27: 100nF, Capacitor_SMD:C_0805_2012Metric_Pad1.18x1.45mm_HandSolder, symbol Device:C
- J10: value Conn_01x05_Pin -> SWD
- J11: value Conn_02x02_2.54 -> UART1
- renumbered C23 to C25, C24 to C26, C28 to C27, C29 to C28, C30 to C29, C31 to C30, C32 to C31, C33 to C32, D14 to D12, D15 to D13, D16 to D14, D17 to D15, D18 to D16, U9 to U10
Connections:
- net VBUS_SENSING: now reaches U10.19 (PB1)
- no-connect marks 9 -> 8
Other:
- moved on the sheet: C25, C26
