File: MCU.kicad_sch (KiCad schematic)
At the start: 37 parts, among them J10 SWD, J11 UART1, SW1 SM5-180UP-1, U10 STM32L072CBT6, Y1 4 MHz, Y2 32768 kHz

Commit message: Dual SIM version
Parts:
- removed L3: MLZ2012M100WT000, Inductor_SMD:L_0805_2012Metric_Pad1.05x1.20mm_HandSolder, symbol Device:L
- D12, D13, D14, D15: value FYLS-0805PGC -> FYLS-0805GC; MPN FYLS-0805PGC -> FYLS-0805GC
- D16: value FYLS-0805URC -> FYLS-0805SRC; MPN FYLS-0805URC -> FYLS-0805SRC
- H1, H2, H3, H4: footprint MountingHole:MountingHole_4.3mm_M4_DIN965_Pad -> MountingHole:MountingHole_3.2mm_M3_Pad_Via
- R30: renamed from R34; value 680 -> 330; MPN RC0805JR-07680RL -> RC0805JR-07330RL
- R31: renamed from R35; value 680 -> 330; MPN RC0805JR-07680RL -> RC0805JR-07330RL
- R32: renamed from R36; value 680 -> 330; MPN RC0805JR-07680RL -> RC0805JR-07330RL
- R33: renamed from R37; value 680 -> 330; MPN RC0805JR-07680RL -> RC0805JR-07330RL
- R35: renamed from R39; value 680 -> 510; MPN RC0805JR-07680RL -> RC0805JR-07510RL
- renumbered R33 to R29, R38 to R34, R40 to R36, R41 to R37, R42 to R38, R43 to R39
Connections:
- net +3V3: now also U10.9 (VDDA)
- net NRST: now also J10.2 (Pin_2); no longer J10.5 (Pin_5)
- net SWCLK: now also J10.5 (Pin_5); no longer J10.2 (Pin_2)

Commit message: Replace SIM800C-DS with A7682E
Parts:
- renumbered C25 to C31, C26 to C32, C27 to C33, C28 to C34, C29 to C35, C30 to C36, C31 to C37, C32 to C38, D12 to D11, D13 to D12, D14 to D13, D15 to D14, D16 to D15, J10 to J11, J11 to J12, R29 to R33, R30 to R34, R31 to R35, R32 to R36, R33 to R37, R34 to R38, R35 to R39, R36 to R40, R37 to R41, R38 to R42, R39 to R43
Connections:
- net UART2_DTR renamed RF_RESET
- net UART2_RI: no longer names the net of U10.39 (PB3)
- no-connect marks 8 -> 9

Commit message: USB connector inversion fix
Parts:
- renumbered C31 to C25, C32 to C26, C33 to C27, C34 to C28, C35 to C29, C36 to C30, C37 to C31, C38 to C32, D15 to D12, D12 to D13, D13 to D14, D14 to D15, D11 to D16, J11 to J10, J12 to J11, R33 to R29, R39 to R30, R35 to R31, R36 to R32, R37 to R33, R38 to R34, R34 to R35, R40 to R36, R41 to R37, R42 to R38, R43 to R39
Connections:
- net LED1: now also R30.1; no longer R35.1
- net LED5: now also R35.1; no longer R30.1
- net UART2_RI: now reaches U10.39 (PB3)
- net RF_RESET renamed UART2_DTR
- no-connect marks 9 -> 8
Other:
- moved on the sheet: D12, D16, R30, R35
