File: RS485.kicad_sch (KiCad schematic)
At the start: 8 parts, among them J7 DG390-5.0-02P, U8 XR3072XIDTR-F

Commit message: Release candidate
Parts:
- JP5: footprint TestPoint:TestPoint_2Pads_Pitch2.54mm_Drill0.8mm -> Connector_PinHeader_2.54mm:PinHeader_1x02_P2.54mm_Vertical
Connections:
- net RS485_P: now also JP5.1 (A); no longer JP5.2 (B)
- net at R26.2: now also JP5.2 (B); no longer JP5.1 (A)
Changed lines of the file:
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@@
 (kicad_sch
-	(version 20260101)
+	(version 20260306)
 	(generator "eeschema")
 	(generator_version "10.0")
@@
 		(lib_id "Jumper:Jumper_2_Open")
 		(at 151.13 90.17 90)
+		(mirror x)
 		(unit 1)
 		(body_style 1)
@@
 		)
 		(property "Value" "Jumper_2_Open"
-			(at 160.02 89.916 90)
-			(show_name no)
-			(do_not_autoplace no)
-			(effects
-				(font
-					(size 1.27 1.27)
-				)
-			)
-		)
-		(property "Footprint" "TestPoint:TestPoint_2Pads_Pitch2.54mm_Drill0.8mm"
+			(at 160.02 90.424 90)
+			(show_name no)
+			(do_not_autoplace no)
+			(effects
+				(font
+					(size 1.27 1.27)
+				)
+			)
+		)
+		(property "Footprint" "Connector_PinHeader_2.54mm:PinHeader_1x02_P2.54mm_Vertical"
 			(at 151.13 90.17 0)
 			(hide yes)

Commit message: Proproduction version
Parts:
- J7: value DG390-5.0-02P -> RS485
- R26: value 680 -> 120; MPN RC0805JR-07680RL -> RC0805JR-07120RL
- renumbered C14 to C16, D11 to D9, U8 to U9
Changed lines of the file:
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@@
 		(dnp no)
 		(fields_autoplaced yes)
-		(property "Reference" "U8"
+		(property "Reference" "U9"
 			(at 124.0633 73.66 0)
 			(show_name no)
@@
 			(project "GSMreceiver"
 				(path "/bbc92722-7b85-49e8-a662-589426df605a/fe2eac04-096c-41cd-9d48-0aafc9873100"
-					(reference "U8")
+					(reference "U9")
 					(unit 1)
 				)
@@
 		(dnp no)
 		(fields_autoplaced yes)
-		(property "Reference" "#PWR034"
+		(property "Reference" "#PWR036"
 			(at 121.92 115.57 0)
 			(hide yes)
@@
 			(project "GSMreceiver"
 				(path "/bbc92722-7b85-49e8-a662-589426df605a/fe2eac04-096c-41cd-9d48-0aafc9873100"
-					(reference "#PWR034")
+					(reference "#PWR036")
 					(unit 1)
 				)
@@
 		(dnp no)
 		(fields_autoplaced yes)
-		(property "Reference" "D11"
+		(property "Reference" "D9"
 			(at 172.72 96.5201 90)
 			(show_name no)
@@
 			(project "GSMreceiver"
 				(path "/bbc92722-7b85-49e8-a662-589426df605a/fe2eac04-096c-41cd-9d48-0aafc9873100"
-					(reference "D11")
+					(reference "D9")
 					(unit 1)
 				)
@@
 			)
 		)
-		(property "Value" "680"
+		(property "Value" "120"
 			(at 154.686 102.87 0)
 			(show_name no)
@@
 			)
 		)
-		(property "MPN" "RC0805JR-07680RL"
+		(property "MPN" "RC0805JR-07120RL"
 			(at 151.13 101.6 0)
 			(hide yes)
@@
 			)
 		)
-		(property "Value" "DG390-5.0-02P"
+		(property "Value" "RS485"
 			(at 213.36 86.3599 0)
 			(show_name no)
@@
 		(dnp no)
 		(fields_autoplaced yes)
-		(property "Reference" "#PWR035"
+		(property "Reference" "#PWR037"
 			(at 181.61 101.6 0)
 			(hide yes)
@@
 			(project "GSMreceiver"
 				(path "/bbc92722-7b85-49e8-a662-589426df605a/fe2eac04-096c-41cd-9d48-0aafc9873100"
-					(reference "#PWR035")
+					(reference "#PWR037")
 					(unit 1)
 				)
@@
 		(in_pos_files yes)
 		(dnp no)
-		(property "Reference" "C14"
+		(property "Reference" "C16"
 			(at 93.726 75.438 0)
 			(show_name no)
@@
 			(project "GSMreceiver"
 				(path "/bbc92722-7b85-49e8-a662-589426df605a/fe2eac04-096c-41cd-9d48-0aafc9873100"
-					(reference "C14")
+					(reference "C16")
 					(unit 1)
 				)
@@
 		(dnp no)
 		(fields_autoplaced yes)
-		(property "Reference" "#PWR033"
+		(property "Reference" "#PWR035"
 			(at 96.52 85.09 0)
 			(hide yes)
@@
 			(project "GSMreceiver"
 				(path "/bbc92722-7b85-49e8-a662-589426df605a/fe2eac04-096c-41cd-9d48-0aafc9873100"
-					(reference "#PWR033")
+					(reference "#PWR035")
 					(unit 1)
 				)
