File: SIMcard.kicad_sch (KiCad schematic)
At the start: 9 parts, among them J8 1042240820

Commit message: Proproduction version
Parts:
- renumbered C15 to C17, C16 to C18, C17 to C19, C18 to C20, D12 to D10
Changed lines of the file:
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@@
 		(dnp no)
 		(fields_autoplaced yes)
-		(property "Reference" "#PWR036"
+		(property "Reference" "#PWR038"
 			(at 111.76 105.41 0)
 			(hide yes)
@@
 			(project "GSMreceiver"
 				(path "/bbc92722-7b85-49e8-a662-589426df605a/0766f5ef-5d4e-4bb3-b73a-d8d6c795d8e3"
-					(reference "#PWR042")
+					(reference "#PWR044")
 					(unit 1)
 				)
 				(path "/bbc92722-7b85-49e8-a662-589426df605a/89f536d0-e840-48e9-a183-c973796594df"
-					(reference "#PWR036")
+					(reference "#PWR038")
 					(unit 1)
 				)
@@
 		(in_pos_files yes)
 		(dnp no)
-		(property "Reference" "#PWR041"
+		(property "Reference" "#PWR043"
 			(at 190.5 93.98 0)
 			(hide yes)
@@
 			(project "GSMreceiver"
 				(path "/bbc92722-7b85-49e8-a662-589426df605a/0766f5ef-5d4e-4bb3-b73a-d8d6c795d8e3"
-					(reference "#PWR047")
+					(reference "#PWR049")
 					(unit 1)
 				)
 				(path "/bbc92722-7b85-49e8-a662-589426df605a/89f536d0-e840-48e9-a183-c973796594df"
-					(reference "#PWR041")
+					(reference "#PWR043")
 					(unit 1)
 				)
@@
 		(in_pos_files yes)
 		(dnp no)
-		(property "Reference" "#PWR040"
+		(property "Reference" "#PWR042"
 			(at 158.75 102.87 0)
 			(hide yes)
@@
 			(project "GSMreceiver"
 				(path "/bbc92722-7b85-49e8-a662-589426df605a/0766f5ef-5d4e-4bb3-b73a-d8d6c795d8e3"
-					(reference "#PWR046")
+					(reference "#PWR048")
 					(unit 1)
 				)
 				(path "/bbc92722-7b85-49e8-a662-589426df605a/89f536d0-e840-48e9-a183-c973796594df"
-					(reference "#PWR040")
+					(reference "#PWR042")
 					(unit 1)
 				)
@@
 		(in_pos_files yes)
 		(dnp no)
-		(property "Reference" "C17"
+		(property "Reference" "C19"
 			(at 152.4 87.122 0)
 			(show_name no)
@@
 			(project "GSMreceiver"
 				(path "/bbc92722-7b85-49e8-a662-589426df605a/0766f5ef-5d4e-4bb3-b73a-d8d6c795d8e3"
-					(reference "C21")
+					(reference "C23")
 					(unit 1)
 				)
 				(path "/bbc92722-7b85-49e8-a662-589426df605a/89f536d0-e840-48e9-a183-c973796594df"
-					(reference "C17")
+					(reference "C19")
 					(unit 1)
 				)
@@
 		(dnp no)
 		(fields_autoplaced yes)
-		(property "Reference" "#PWR037"
+		(property "Reference" "#PWR039"
 			(at 135.89 66.04 0)
 			(hide yes)
@@
 			(project "GSMreceiver"
 				(path "/bbc92722-7b85-49e8-a662-589426df605a/0766f5ef-5d4e-4bb3-b73a-d8d6c795d8e3"
-					(reference "#PWR043")
+					(reference "#PWR045")
 					(unit 1)
 				)
 				(path "/bbc92722-7b85-49e8-a662-589426df605a/89f536d0-e840-48e9-a183-c973796594df"
-					(reference "#PWR037")
+					(reference "#PWR039")
 					(unit 1)
 				)
@@
 		(in_pos_files yes)
 		(dnp no)
-		(property "Reference" "C15"
+		(property "Reference" "C17"
 			(at 119.888 63.5 90)
 			(show_name no)
@@
 			(project "GSMreceiver"
 				(path "/bbc92722-7b85-49e8-a662-589426df605a/0766f5ef-5d4e-4bb3-b73a-d8d6c795d8e3"
-					(reference "C19")
+					(reference "C21")
 					(unit 1)
 				)
 				(path "/bbc92722-7b85-49e8-a662-589426df605a/89f536d0-e840-48e9-a183-c973796594df"
-					(reference "C15")
+					(reference "C17")
 					(unit 1)
 				)
@@
 		(in_pos_files yes)
 		(dnp no)
-		(property "Reference" "C16"
+		(property "Reference" "C18"
 			(at 143.51 87.376 0)
 			(show_name no)
@@
 			(project "GSMreceiver"
 				(path "/bbc92722-7b85-49e8-a662-589426df605a/0766f5ef-5d4e-4bb3-b73a-d8d6c795d8e3"
-					(reference "C20")
+					(reference "C22")
 					(unit 1)
 				)
 				(path "/bbc92722-7b85-49e8-a662-589426df605a/89f536d0-e840-48e9-a183-c973796594df"
-					(reference "C16")
+					(reference "C18")
 					(unit 1)
 				)
@@
 		(dnp no)
 		(fields_autoplaced yes)
-		(property "Reference" "D12"
+		(property "Reference" "D10"
 			(at 120.65 90.1699 0)
 			(show_name no)
@@
 			(project "GSMreceiver"
 				(path "/bbc92722-7b85-49e8-a662-589426df605a/0766f5ef-5d4e-4bb3-b73a-d8d6c795d8e3"
-					(reference "D13")
+					(reference "D11")
 					(unit 1)
 				)
 				(path "/bbc92722-7b85-49e8-a662-589426df605a/89f536d0-e840-48e9-a183-c973796594df"
-					(reference "D12")
+					(reference "D10")
 					(unit 1)
 				)
@@
 		(in_pos_files yes)
 		(dnp no)
-		(property "Reference" "#PWR039"
+		(property "Reference" "#PWR041"
 			(at 149.86 102.87 0)
 			(hide yes)
@@
 			(project "GSMreceiver"
 				(path "/bbc92722-7b85-49e8-a662-589426df605a/0766f5ef-5d4e-4bb3-b73a-d8d6c795d8e3"
-					(reference "#PWR045")
+					(reference "#PWR047")
 					(unit 1)
 				)
 				(path "/bbc92722-7b85-49e8-a662-589426df605a/89f536d0-e840-48e9-a183-c973796594df"
-					(reference "#PWR039")
+					(reference "#PWR041")
 					(unit 1)
 				)
@@
 		(in_pos_files yes)
 		(dnp no)
-		(property "Reference" "C18"
+		(property "Reference" "C20"
 			(at 161.29 87.122 0)
 			(show_name no)
@@
 			(project "GSMreceiver"
 				(path "/bbc92722-7b85-49e8-a662-589426df605a/0766f5ef-5d4e-4bb3-b73a-d8d6c795d8e3"
-					(reference "C22")
+					(reference "C24")
 					(unit 1)
 				)
 				(path "/bbc92722-7b85-49e8-a662-589426df605a/89f536d0-e840-48e9-a183-c973796594df"
-					(reference "C18")
+					(reference "C20")
 					(unit 1)
 				)
@@
 		(in_pos_files yes)
 		(dnp no)
-		(property "Reference" "#PWR038"
+		(property "Reference" "#PWR040"
 			(at 140.97 102.87 0)
 			(hide yes)
@@
 			(project "GSMreceiver"
 				(path "/bbc92722-7b85-49e8-a662-589426df605a/0766f5ef-5d4e-4bb3-b73a-d8d6c795d8e3"
-					(reference "#PWR044")
+					(reference "#PWR046")
 					(unit 1)
 				)
 				(path "/bbc92722-7b85-49e8-a662-589426df605a/89f536d0-e840-48e9-a183-c973796594df"
-					(reference "#PWR038")
-					(unit 1)
-				)
+					(reference "#PWR040")
+					(unit 1)
+				)
