File: GSMreceiver.kicad_pcb (KiCad board)
At the start: 2 copper layers, 69 x 83 mm, 159 parts, among them J1 Relay_1, J10 1042240820, J11 SWD, J12 UART1, J13 DG390-5.0-02P, J2 Relay_2, J3 Relay_3, J4 Relay_4, J5 USB_RF, J6 RF Antenna, J7 USB-C, J8 RS485, J9 1042240820, Q1 MUN5233DW1, SW1 SM5-180UP-1, U1 PRAB34S, U10 STM32L072CBT6, U2 PRAB34S, U3 PRAB34S, U4 PRAB34S, U5 AP63203WU, U6 AP63200WU, U7 A7682E, U8 USBLC6-2SC6, U9 XR3072XIDTR-F, Y1 4 MHz, Y2 32768 kHz

Commit message: Silk update
Parts:
- moved JP6 35.7 mm to (87.0, 36.1)
- moved FID5 3.16 mm to (46.0, 38.0)
- moved R40 1.22 mm to (45.4, 61.1)
- moved R32 1.20 mm to (40.7, 58.0)
- moved FID1 1.00 mm to (46.0, 38.0)
- moved C41 0.90 mm to (83.9, 84.9)
- moved C10 0.40 mm to (54.1, 28.6)
- moved C37 0.10 mm to (55.5, 64.6)
- moved C8 0.10 mm to (74.4, 50.9)
- moved C9 0.10 mm to (74.4, 48.1)
- moved C15 0.10 mm to (69.9, 40.6)
- moved C19 0.05 mm to (64.6, 29.9)
Routing:
- net Net-(JP6-B): track 39.5 -> 44.1 mm
- net /RFmodule/SIM2_RST: track 18.0 -> 21.5 mm
- net /MCU/TAMPER: track 49.9 -> 47.1 mm
- net /MCU/NRST: track 29.2 -> 26.6 mm
- net /RFmodule/SIM2_CLK: track 13.9 -> 15.8 mm
- net GNDD: track 16.2 -> 14.5 mm, vias 83 -> 82
- net /SIMcard2/CARD_RST: track 11.4 -> 10.2 mm
- net /RS485_EN: track 43.1 -> 41.9 mm
- net +3V3: track 37.4 -> 38.1 mm
- net /MCU/SWDIO: track 11.9 -> 12.4 mm
- net /MCU/SWCLK: track 20.2 -> 20.7 mm

Commit message: C37
Parts:
- moved C31 1.08 mm to (52.4, 59.8), turned to 180 degrees
Routing:
- net +3V3: track 38.1 -> 37.5 mm
- net GNDD: vias 82 -> 83
Changed lines of the file:
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@@
 	(footprint "Capacitor_SMD:C_0805_2012Metric_Pad1.18x1.45mm_HandSolder"
 		(layer "B.Cu")
-		(at 51.4 59.4 90)
+		(at 52.4 59.8 180)
 		(descr "Capacitor SMD 0805 (2012 Metric), square (rectangular) end terminal, IPC-7351 nominal with elongated pad for handsoldering. (Body size source: IPC-SM-782 page 76, https://www.pcb-3d.com/wordpress/wp-content/uploads/ipc-sm-782a_amendment_1_and_2.pdf, https://docs.google.com/spreadsheets/d/1BsfQQcO9C6DZCsRaXUlFlo91Tg2WpOkGARC1WS5S8t0/edit?usp=sharing), generated with kicad-footprint-generator")
 		(tags "capacitor handsolder")
 		(property "Reference" "C31"
-			(at -0.1 1.8 90)
+			(at -0.1 1.8 0)
 			(layer "B.SilkS")
 			(effects
@@
 		)
 		(property "Value" "100nF"
-			(at 0 -1.68 90)
+			(at 0 -1.68 0)
 			(layer "B.Fab")
 			(effects
@@
 		)
 		(property "Datasheet" ""
-			(at 0 0 90)
+			(at 0 0 0)
 			(layer "B.Fab")
 			(hide yes)
@@
 		)
 		(property "Description" "Unpolarized capacitor"
-			(at 0 0 90)
+			(at 0 0 0)
 			(layer "B.Fab")
 			(hide yes)
@@
 		)
 		(property "Manufacturer" "YAGEO"
-			(at 0 0 270)
+			(at 0 0 0)
 			(unlocked yes)
 			(layer "B.Fab")
@@
 		)
 		(property "MPN" "CC0805KRX7R8BB104"
-			(at 0 0 270)
+			(at 0 0 0)
 			(unlocked yes)
 			(layer "B.Fab")
@@
 		(duplicate_pad_numbers_are_jumpers no)
 		(fp_line
-			(start -0.261252 -0.735)
-			(end 0.261252 -0.735)
+			(start -0.261252 0.735)
+			(end 0.261252 0.735)
 			(stroke
 				(width 0.12)
@@
 		)
 		(fp_line
-			(start -0.261252 0.735)
-			(end 0.261252 0.735)
+			(start -0.261252 -0.735)
+			(end 0.261252 -0.735)
 			(stroke
 				(width 0.12)
@@
 		)
 		(fp_text user "${REFERENCE}"
-			(at 0 0 90)
+			(at 0 0 0)
 			(layer "B.Fab")
 			(effects
@@
 		)
 		(pad "1" smd roundrect
-			(at -1.0375 0 90)
+			(at -1.0375 0 180)
 			(size 1.175 1.45)
 			(layers "B.Cu" "B.Mask" "B.Paste")
@@
 		)
 		(pad "2" smd roundrect
-			(at 1.0375 0 90)
+			(at 1.0375 0 180)
 			(size 1.175 1.45)
 			(layers "B.Cu" "B.Mask" "B.Paste")
@@
 	)
 	(via
+		(at 45.7 58.6)
+		(size 1)
+		(drill 0.4)
+		(layers "F.Cu" "B.Cu")
+		(capping no)
+		(covering
+			(front no)
+			(back no)
+		)
+		(plugging
+			(front no)
+			(back no)
+		)
+		(filling no)
+		(net "GNDD")
+	)
+	(via
 		(at 86.2 46.9)
 		(size 1)
@@
 	)
 	(segment
+		(start 51.3425 59.82)
+		(end 51.3625 59.8)
+		(width 0.6)
+		(layer "B.Cu")
+		(net "+3V3")
+	)
+	(segment
 		(start 68.3625 69.45)
 		(end 69.9 69.45)
@@
 	)
 	(segment
-		(start 51.4 58.3625)
-		(end 49.4575 58.3625)
-		(width 0.6)
-		(layer "B.Cu")
-		(net "+3V3")
-	)
-	(segment
-		(start 49.4575 58.3625)
-		(end 48 59.82)
+		(start 48 59.82)
+		(end 51.3425 59.82)
 		(width 0.6)
 		(layer "B.Cu")
